File: AmigaExternalBoard.sch (KiCad schematic (older format))
At the start: 14 parts, among them J1 Conn_01x24, J2 Conn_01x24, J3 Conn_01x24, SW1 SW_SPDT, SW2 SW_SPDT, SW3 SW_SPDT

Commit message: Modified   AmigaExternalBoard.kicad_pcb Modified   AmigaExternalBoard.kicad_pcb-bak Modified   AmigaExternalBoard.sch Modified   AmigaExternalBoard.sch-bak
Parts:
- R1, R3: value R -> R-OptionalPullup-SCL
- R2, R4: value R -> R-OptionalPullup-SDA
Changed lines of the file:
@@
 P 4400 3750
 F 0 "R1" H 4470 3796 50  0000 L CNN
-F 1 "R" H 4470 3705 50  0000 L CNN
+F 1 "R-OptionalPullup-SCL" V 4400 3950 50  0000 L CNN
 F 2 "Resistor_THT:R_Axial_DIN0207_L6.3mm_D2.5mm_P10.16mm_Horizontal" V 4330 3750 50  0001 C CNN
 F 3 "~" H 4400 3750 50  0001 C CNN
@@
 P 4150 3750
 F 0 "R2" H 4220 3796 50  0000 L CNN
-F 1 "R" H 4220 3705 50  0000 L CNN
+F 1 "R-OptionalPullup-SDA" V 4150 3950 50  0000 L CNN
 F 2 "Resistor_THT:R_Axial_DIN0207_L6.3mm_D2.5mm_P10.16mm_Horizontal" V 4080 3750 50  0001 C CNN
 F 3 "~" H 4150 3750 50  0001 C CNN
@@
 P 3900 3750
 F 0 "R3" H 3970 3796 50  0000 L CNN
-F 1 "R" H 3970 3705 50  0000 L CNN
+F 1 "R-OptionalPullup-SCL" V 3900 3950 50  0000 L CNN
 F 2 "Resistor_SMD:R_0805_2012Metric_Pad1.15x1.40mm_HandSolder" V 3830 3750 50  0001 C CNN
 F 3 "~" H 3900 3750 50  0001 C CNN
@@
 P 3650 3750
 F 0 "R4" H 3720 3796 50  0000 L CNN
-F 1 "R" H 3720 3705 50  0000 L CNN
+F 1 "R-OptionalPullup-SDA" V 3650 3950 50  0000 L CNN
 F 2 "Resistor_SMD:R_0805_2012Metric_Pad1.15x1.40mm_HandSolder" V 3580 3750 50  0001 C CNN
 F 3 "~" H 3650 3750 50  0001 C CNN

Commit message: Modified   AmigaExternalBoard-cache.lib Modified   AmigaExternalBoard.kicad_pcb Modified   AmigaExternalBoard.kicad_pcb-bak Modified   AmigaExternalBoard.sch Modified   AmigaExternalBoard.sch-bak Modified   fp-info-cache Added      bom/ibom.html
Parts:
- added JP1, JP2: Jumper_3_Open, DCDModules:SolderJumper-3_P0.5mm_Open_Pad0.5x0.5mm, symbol Jumper:Jumper_3_Open
Connections:
- net +3V3: now also JP1.1 (A), JP2.1 (A); no longer DSP1.2 (VCC)
- net GND: now also JP1.3 (B), JP2.3 (B); no longer DSP1.1 (GND)
- net GotekBTN1: now reaches J1.20 (Pin_20)
- net GotekBTN1: now also J2.4 (Pin_4), J3.5 (Pin_5)
- net GotekBTN2: now reaches J1.21 (Pin_21)
- net GotekBTN2: now also J2.3 (Pin_3), J3.4 (Pin_4)
- net GotekLED: now reaches J1.22 (Pin_22)
- net GotekLED: now also J2.2 (Pin_2), J3.3 (Pin_3)
- new net: DSP1.1 (GND), JP1.2 (C)
- new net: DSP1.2 (VCC), JP2.2 (C)
Other:
- moved on the sheet: SW1, SW2, SW3
Changed lines of the file:
@@
 L power:+3V3 #PWR0110
 U 1 1 608DF8E7
-P 7400 2150
-F 0 "#PWR0110" H 7400 2000 50  0001 C CNN
-F 1 "+3V3" V 7415 2278 50  0000 L CNN
-F 2 "" H 7400 2150 50  0001 C CNN
-F 3 "" H 7400 2150 50  0001 C CNN
-	1    7400 2150
-	0    1    1    0
+P 7050 1700
+F 0 "#PWR0110" H 7050 1550 50  0001 C CNN
+F 1 "+3V3" V 7065 1828 50  0000 L CNN
+F 2 "" H 7050 1700 50  0001 C CNN
+F 3 "" H 7050 1700 50  0001 C CNN
+	1    7050 1700
+	0    -1   -1   0
 $EndComp
 $Comp
 L power:GND #PWR0111
 U 1 1 608DFB7F
-P 7400 2050
-F 0 "#PWR0111" H 7400 1800 50  0001 C CNN
-F 1 "GND" V 7405 1922 50  0000 R CNN
-F 2 "" H 7400 2050 50  0001 C CNN
-F 3 "" H 7400 2050 50  0001 C CNN
-	1    7400 2050
-	0    -1   -1   0
-$EndComp
-Wire Wire Line
-	7400 2050 7300 2050
-Wire Wire Line
-	7400 2150 7300 2150
+P 7750 1700
+F 0 "#PWR0111" H 7750 1450 50  0001 C CNN
+F 1 "GND" V 7755 1572 50  0000 R CNN
+F 2 "" H 7750 1700 50  0001 C CNN
+F 3 "" H 7750 1700 50  0001 C CNN
+	1    7750 1700
+	0    -1   -1   0
+$EndComp
+Wire Wire Line
+	7750 1700 7650 1700
+Wire Wire Line
+	7050 1700 7150 1700
 Text GLabel 7600 2350 2    50   Input ~ 0
 SDA(DSP)
@@
 L Switch:SW_SPDT SW1
 U 1 1 60849D99
-P 9000 850
-F 0 "SW1" H 9000 1135 50  0000 C CNN
-F 1 "SW_SPDT" H 9000 1044 50  0000 C CNN
-F 2 "Button_Switch_THT:SW_CuK_OS102011MA1QN1_SPDT_Angled" H 9000 850 50  0001 C CNN
-F 3 "~" H 9000 850 50  0001 C CNN
-	1    9000 850
+P 10100 950
+F 0 "SW1" H 10100 1235 50  0000 C CNN
+F 1 "SW_SPDT" H 10100 1144 50  0000 C CNN
+F 2 "Button_Switch_THT:SW_CuK_OS102011MA1QN1_SPDT_Angled" H 10100 950 50  0001 C CNN
+F 3 "~" H 10100 950 50  0001 C CNN
+	1    10100 950
 	1    0    0    -1
 $EndComp
@@
 L Switch:SW_SPDT SW2
 U 1 1 6084A881
-P 9000 1350
-F 0 "SW2" H 9000 1635 50  0000 C CNN
-F 1 "SW_SPDT" H 9000 1544 50  0000 C CNN
-F 2 "Button_Switch_THT:SW_CuK_OS102011MA1QN1_SPDT_Angled" H 9000 1350 50  0001 C CNN
-F 3 "~" H 9000 1350 50  0001 C CNN
-	1    9000 1350
+P 10100 1450
+F 0 "SW2" H 10100 1735 50  0000 C CNN
+F 1 "SW_SPDT" H 10100 1644 50  0000 C CNN
+F 2 "Button_Switch_THT:SW_CuK_OS102011MA1QN1_SPDT_Angled" H 10100 1450 50  0001 C CNN
+F 3 "~" H 10100 1450 50  0001 C CNN
+	1    10100 1450
 	1    0    0    -1
 $EndComp
@@
 L Switch:SW_SPDT SW3
 U 1 1 6084B3F7
-P 9000 1850
-F 0 "SW3" H 9000 2135 50  0000 C CNN
-F 1 "SW_SPDT" H 9000 2044 50  0000 C CNN
-F 2 "Button_Switch_THT:SW_CuK_OS102011MA1QN1_SPDT_Angled" H 9000 1850 50  0001 C CNN
-F 3 "~" H 9000 1850 50  0001 C CNN
-	1    9000 1850
-	1    0    0    -1
-$EndComp
-Text GLabel 8700 850  0    50   Input ~ 0
+P 10100 1950
+F 0 "SW3" H 10100 2235 50  0000 C CNN
+F 1 "SW_SPDT" H 10100 2144 50  0000 C CNN
+F 2 "Button_Switch_THT:SW_CuK_OS102011MA1QN1_SPDT_Angled" H 10100 1950 50  0001 C CNN
+F 3 "~" H 10100 1950 50  0001 C CNN
+	1    10100 1950
+	1    0    0    -1
+$EndComp
+Text GLabel 9800 950  0    50   Input ~ 0
 SW1_2
-Text GLabel 9300 750  2    50   Input ~ 0
+Text GLabel 10400 850  2    50   Input ~ 0
 SW1_1
-Text GLabel 9300 950  2    50   Input ~ 0
+Text GLabel 10400 1050 2    50   Input ~ 0
 SW1_3
 Wire Wire Line
-	9200 750  9300 750
-Wire Wire Line
-	9200 950  9300 950
-Wire Wire Line
-	8800 850  8700 850
-Text GLabel 8700 1350 0    50   Input ~ 0
+	10300 850  10400 850
+Wire Wire Line
+	10300 1050 10400 1050
+Wire Wire Line
+	9900 950  9800 950
+Text GLabel 9800 1450 0    50   Input ~ 0
 SW2_2
 Wire Wire Line
-	8800 1350 8700 1350
-Text GLabel 8700 1850 0    50   Input ~ 0
+	9900 1450 9800 1450
+Text GLabel 9800 1950 0    50   Input ~ 0
 SW3_2
 Wire Wire Line
-	8800 1850 8700 1850
-Text GLabel 9300 1250 2    50   Input ~ 0
+	9900 1950 9800 1950
+Text GLabel 10400 1350 2    50   Input ~ 0
 SW2_1
-Text GLabel 9300 1450 2    50   Input ~ 0
+Text GLabel 10400 1550 2    50   Input ~ 0
 SW2_3
 Wire Wire Line
-	9200 1250 9300 1250
-Wire Wire Line
-	9200 1450 9300 1450
-Text GLabel 9300 1750 2    50   Input ~ 0
+	10300 1350 10400 1350
+Wire Wire Line
+	10300 1550 10400 1550
+Text GLabel 10400 1850 2    50   Input ~ 0
 SW3_1
-Text GLabel 9300 1950 2    50   Input ~ 0
+Text GLabel 10400 2050 2    50   Input ~ 0
 SW3_3
 Wire Wire Line
-	9200 1750 9300 1750
-Wire Wire Line
-	9200 1950 9300 1950
+	10300 1850 10400 1850
+Wire Wire Line
+	10300 2050 10400 2050
 Text GLabel 1650 2200 2    50   Input ~ 0
 SW1_2
@@
 Text GLabel 5000 1700 0    50   Input ~ 0
 SW3_1
+Text GLabel 5000 1400 0    50   Input ~ 0
+GotekBTN1
+Text GLabel 5000 1300 0    50   Input ~ 0
+GotekBTN2
+Text GLabel 5000 1200 0    50   Input ~ 0
+GotekLED
+Wire Wire Line
+	5000 1400 5300 1400
+Wire Wire Line
+	5000 1300 5300 1300
+Wire Wire Line
+	5000 1200 5300 1200
+Text GLabel 3400 1400 2    50   Input ~ 0
+GotekBTN1
+Text GLabel 3400 1300 2    50   Input ~ 0
+GotekBTN2
+Text GLabel 3400 1200 2    50   Input ~ 0
+GotekLED
+Wire Wire Line
+	3400 1400 3100 1400
+Wire Wire Line
+	3400 1300 3100 1300
+Wire Wire Line
+	3400 1200 3100 1200
+Text GLabel 1650 3000 2    50   Input ~ 0
+GotekBTN1
+Text GLabel 1650 3100 2    50   Input ~ 0
+GotekBTN2
+Text GLabel 1650 3200 2    50   Input ~ 0
+GotekLED
+Wire Wire Line
+	1650 3000 1350 3000
+Wire Wire Line
+	1650 3100 1350 3100
+Wire Wire Line
+	1650 3200 1350 3200
+$Comp
+L Jumper:Jumper_3_Open JP1
+U 1 1 612AA9FC
+P 7400 1700
+F 0 "JP1" H 7400 1924 50  0000 C CNN
+F 1 "Jumper_3_Open" H 7400 1833 50  0000 C CNN
+F 2 "DCDModules:SolderJumper-3_P0.5mm_Open_Pad0.5x0.5mm" H 7400 1700 50  0001 C CNN
+F 3 "~" H 7400 1700 50  0001 C CNN
+	1    7400 1700
+	1    0    0    -1
+$EndComp
+Wire Wire Line
+	7300 2050 7400 2050
+Wire Wire Line
+	7400 2050 7400 1850
+$Comp
+L power:+3V3 #PWR01
+U 1 1 612CB19F
+P 7750 1350
+F 0 "#PWR01" H 7750 1200 50  0001 C CNN
+F 1 "+3V3" V 7765 1478 50  0000 L CNN
+F 2 "" H 7750 1350 50  0001 C CNN
+F 3 "" H 7750 1350 50  0001 C CNN
+	1    7750 1350
+	0    -1   -1   0
+$EndComp
+$Comp
+L power:GND #PWR02
+U 1 1 612CB1D3
+P 8450 1350
+F 0 "#PWR02" H 8450 1100 50  0001 C CNN
+F 1 "GND" V 8455 1222 50  0000 R CNN
+F 2 "" H 8450 1350 50  0001 C CNN
+F 3 "" H 8450 1350 50  0001 C CNN
+	1    8450 1350
+	0    -1   -1   0
+$EndComp
+Wire Wire Line
+	8450 1350 8350 1350
+Wire Wire Line
+	7750 1350 7850 1350
+$Comp
+L Jumper:Jumper_3_Open JP2
+U 1 1 612CB1DF
+P 8100 1350
+F 0 "JP2" H 8100 1574 50  0000 C CNN
+F 1 "Jumper_3_Open" H 8100 1483 50  0000 C CNN
+F 2 "DCDModules:SolderJumper-3_P0.5mm_Open_Pad0.5x0.5mm" H 8100 1350 50  0001 C CNN
+F 3 "~" H 8100 1350 50  0001 C CNN
+	1    8100 1350
+	1    0    0    -1
+$EndComp
+Wire Wire Line
+	7300 2150 8100 2150
+Wire Wire Line
+	8100 2150 8100 1500
 $EndSCHEMATC
