File: AmigaExternalBoard.kicad_pcb (KiCad board)
At the start: 2 copper layers, 132.9 x 40.7 mm, 22 parts, among them J1 Conn_01x24, J2 Conn_01x24, J3 Conn_01x24, SW1 SW_SPDT, SW2 SW_SPDT, SW3 SW_SPDT

Commit message: Modified   AmigaExternalBoard.kicad_pcb Modified   AmigaExternalBoard.kicad_pcb-bak Modified   AmigaExternalBoard.sch Modified   AmigaExternalBoard.sch-bak
Parts:
- R1, R3: value R -> R-OptionalPullup-SCL
- R2, R4: value R -> R-OptionalPullup-SDA

Commit message: Modified   AmigaExternalBoard-cache.lib Modified   AmigaExternalBoard.kicad_pcb Modified   AmigaExternalBoard.kicad_pcb-bak Modified   AmigaExternalBoard.sch Modified   AmigaExternalBoard.sch-bak Modified   fp-info-cache Added      bom/ibom.html
Parts:
- added JP1: Jumper_3_Open, DCDModules:SolderJumper-3_P0.5mm_Open_Pad0.5x0.5mm, F.Cu at (100.4, 58.1)
- added JP2: Jumper_3_Open, DCDModules:SolderJumper-3_P0.5mm_Open_Pad0.5x0.5mm, F.Cu at (102.9, 58.1)
Connections:
- DSP1 pad 1: GND -> Net-(DSP1-Pad1)
- DSP1 pad 2: +3V3 -> Net-(DSP1-Pad2)
- J1 pad 20: Net-(J1-Pad20) -> GotekBTN1
- J1 pad 21: Net-(J1-Pad21) -> GotekBTN2
- J1 pad 22: Net-(J1-Pad22) -> GotekLED
- J2 pad 2: Net-(J2-Pad2) -> GotekLED
- J2 pad 3: Net-(J2-Pad3) -> GotekBTN2
- J2 pad 4: Net-(J2-Pad4) -> GotekBTN1
- J3 pad 3: Net-(J3-Pad3) -> GotekLED
- J3 pad 4: Net-(J3-Pad4) -> GotekBTN2
- J3 pad 5: Net-(J3-Pad5) -> GotekBTN1
Routing:
- net GotekBTN2: track 0.00 -> 26.6 mm
- net GotekLED: track 0.00 -> 24.0 mm
- net GotekBTN1: track 0.00 -> 23.3 mm
- net Net-(DSP1-Pad1): track 0.00 -> 2.33 mm
- net Net-(DSP1-Pad2): track 0.00 -> 2.33 mm
- net +3V3: track 96.6 -> 98.9 mm, vias 1 -> 2
- net SW3_3: track 67.6 -> 66.9 mm
Other:
- board text added: "+3V3"
- board text added: "JB0 (+)"
- board text added: "SW3_2"
- board text removed: "+"
- board text removed: "JB0"
